File: enclosure/switch/switch.sch (EAGLE design)
At the start: 10 parts, among them SW1 TVGP01-G73BB

Commit message: [update] brdを作製
Connections:
- net +3V3: now also U$1.1; no longer U$1.2
- net +5V: now also U$1.2; no longer U$1.1
- net GND: now also U$1.3; no longer U$1.8
- net N$3: now also U$1.6; no longer U$1.7
- net N$4: now also U$1.5; no longer U$1.6
- net N$5: now also U$1.7; no longer U$1.5
- net N$6: now also U$1.8; no longer U$1.3
Other:
- moved on the sheet: LED2, R2
Changed lines of the file:
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@@
 </variantdefs>
 <classes>
-<class number="0" name="default" width="0" drill="0">
+<class number="0" name="default" width="0.508" drill="0">
+</class>
+<class number="1" name="Power" width="1.016" drill="0">
 </class>
 </classes>
@@
 <instance part="U$2" gate="G$1" x="38.1" y="53.34" rot="R270"/>
 <instance part="LED1" gate="G$1" x="55.88" y="30.48" rot="R90"/>
-<instance part="LED2" gate="G$1" x="55.88" y="17.78" rot="R90"/>
+<instance part="LED2" gate="G$1" x="55.88" y="20.32" rot="R90"/>
 <instance part="R1" gate="G$1" x="43.18" y="30.48"/>
-<instance part="R2" gate="G$1" x="43.18" y="17.78"/>
+<instance part="R2" gate="G$1" x="43.18" y="20.32"/>
 <instance part="GND1" gate="1" x="66.04" y="25.4"/>
-<instance part="GND2" gate="1" x="66.04" y="12.7"/>
-<instance part="GND3" gate="1" x="12.7" y="5.08"/>
-<instance part="P+1" gate="1" x="7.62" y="40.64"/>
+<instance part="GND2" gate="1" x="66.04" y="15.24"/>
+<instance part="GND3" gate="1" x="30.48" y="2.54"/>
+<instance part="P+1" gate="1" x="15.24" y="40.64"/>
 <instance part="P+2" gate="1" x="50.8" y="66.04"/>
-<instance part="+3V1" gate="G$1" x="15.24" y="40.64"/>
+<instance part="+3V1" gate="G$1" x="7.62" y="40.64"/>
 <instance part="+3V2" gate="G$1" x="78.74" y="66.04"/>
 <instance part="U$1" gate="G$1" x="-5.08" y="20.32" rot="R270"/>
@@
 </busses>
 <nets>
-<net name="+5V" class="0">
-<segment>
-<pinref part="U$1" gate="G$1" pin="1"/>
-<pinref part="P+1" gate="1" pin="+5V"/>
-<wire x1="0" y1="29.21" x2="7.62" y2="29.21" width="0.1524" layer="91"/>
-<wire x1="7.62" y1="29.21" x2="7.62" y2="38.1" width="0.1524" layer="91"/>
-</segment>
+<net name="+5V" class="1">
 <segment>
 <pinref part="U$2" gate="G$1" pin="2"/>
@@
 <wire x1="50.8" y1="53.34" x2="50.8" y2="63.5" width="0.1524" layer="91"/>
 </segment>
-</net>
-<net name="+3V3" class="0">
 <segment>
 <pinref part="U$1" gate="G$1" pin="2"/>
-<pinref part="+3V1" gate="G$1" pin="+3V3"/>
+<pinref part="P+1" gate="1" pin="+5V"/>
 <wire x1="0" y1="26.67" x2="15.24" y2="26.67" width="0.1524" layer="91"/>
 <wire x1="15.24" y1="26.67" x2="15.24" y2="38.1" width="0.1524" layer="91"/>
 </segment>
+</net>
+<net name="+3V3" class="1">
 <segment>
 <pinref part="+3V2" gate="G$1" pin="+3V3"/>
@@
 <wire x1="20.32" y1="68.58" x2="20.32" y2="71.12" width="0.1524" layer="91"/>
 </segment>
-</net>
-<net name="GND" class="0">
-<segment>
-<pinref part="U$1" gate="G$1" pin="8"/>
-<pinref part="GND3" gate="1" pin="GND"/>
-<wire x1="0" y1="11.43" x2="12.7" y2="11.43" width="0.1524" layer="91"/>
-<wire x1="12.7" y1="11.43" x2="12.7" y2="7.62" width="0.1524" layer="91"/>
-</segment>
+<segment>
+<pinref part="U$1" gate="G$1" pin="1"/>
+<pinref part="+3V1" gate="G$1" pin="+3V3"/>
+<wire x1="0" y1="29.21" x2="7.62" y2="29.21" width="0.1524" layer="91"/>
+<wire x1="7.62" y1="29.21" x2="7.62" y2="38.1" width="0.1524" layer="91"/>
+</segment>
+</net>
+<net name="GND" class="1">
 <segment>
 <pinref part="GND2" gate="1" pin="GND"/>
-<wire x1="66.04" y1="17.78" x2="66.04" y2="15.24" width="0.1524" layer="91"/>
+<wire x1="66.04" y1="20.32" x2="66.04" y2="17.78" width="0.1524" layer="91"/>
 <pinref part="LED2" gate="G$1" pin="C"/>
-<wire x1="60.96" y1="17.78" x2="66.04" y2="17.78" width="0.1524" layer="91"/>
+<wire x1="60.96" y1="20.32" x2="66.04" y2="20.32" width="0.1524" layer="91"/>
 </segment>
 <segment>
@@
 <wire x1="5.08" y1="54.61" x2="5.08" y2="50.8" width="0.1524" layer="91"/>
 </segment>
-</net>
-<net name="N$3" class="0">
-<segment>
-<pinref part="R2" gate="G$1" pin="1"/>
-<pinref part="U$1" gate="G$1" pin="7"/>
-<wire x1="38.1" y1="17.78" x2="38.1" y2="13.97" width="0.1524" layer="91"/>
-<wire x1="38.1" y1="13.97" x2="0" y2="13.97" width="0.1524" layer="91"/>
+<segment>
+<pinref part="U$1" gate="G$1" pin="3"/>
+<pinref part="GND3" gate="1" pin="GND"/>
+<wire x1="0" y1="24.13" x2="30.48" y2="24.13" width="0.1524" layer="91"/>
+<wire x1="30.48" y1="24.13" x2="30.48" y2="5.08" width="0.1524" layer="91"/>
 </segment>
 </net>
@@
 <pinref part="R1" gate="G$1" pin="1"/>
 <wire x1="38.1" y1="30.48" x2="35.56" y2="30.48" width="0.1524" layer="91"/>
-<pinref part="U$1" gate="G$1" pin="6"/>
-<wire x1="35.56" y1="30.48" x2="35.56" y2="16.51" width="0.1524" layer="91"/>
-<wire x1="35.56" y1="16.51" x2="0" y2="16.51" width="0.1524" layer="91"/>
+<wire x1="35.56" y1="30.48" x2="33.02" y2="30.48" width="0.1524" layer="91"/>
+<pinref part="U$1" gate="G$1" pin="5"/>
+<wire x1="0" y1="19.05" x2="20.32" y2="19.05" width="0.1524" layer="91"/>
+<wire x1="20.32" y1="19.05" x2="20.32" y2="30.48" width="0.1524" layer="91"/>
+<wire x1="20.32" y1="30.48" x2="33.02" y2="30.48" width="0.1524" layer="91"/>
 </segment>
 </net>
@@
 <pinref part="LED2" gate="G$1" pin="A"/>
 <pinref part="R2" gate="G$1" pin="2"/>
-<wire x1="53.34" y1="17.78" x2="48.26" y2="17.78" width="0.1524" layer="91"/>
+<wire x1="53.34" y1="20.32" x2="48.26" y2="20.32" width="0.1524" layer="91"/>
 </segment>
 </net>
@@
 <pinref part="SW1" gate="G$1" pin="1"/>
 <wire x1="91.44" y1="53.34" x2="93.98" y2="53.34" width="0.1524" layer="91"/>
-<pinref part="U$1" gate="G$1" pin="5"/>
 <wire x1="93.98" y1="53.34" x2="96.52" y2="53.34" width="0.1524" layer="91"/>
-<wire x1="0" y1="19.05" x2="33.02" y2="19.05" width="0.1524" layer="91"/>
-<wire x1="33.02" y1="19.05" x2="33.02" y2="35.56" width="0.1524" layer="91"/>
-<wire x1="33.02" y1="35.56" x2="93.98" y2="35.56" width="0.1524" layer="91"/>
-<wire x1="93.98" y1="35.56" x2="93.98" y2="53.34" width="0.1524" layer="91"/>
 <junction x="93.98" y="53.34"/>
+<pinref part="U$1" gate="G$1" pin="7"/>
+<wire x1="93.98" y1="38.1" x2="93.98" y2="53.34" width="0.1524" layer="91"/>
+<wire x1="0" y1="13.97" x2="25.4" y2="13.97" width="0.1524" layer="91"/>
+<wire x1="25.4" y1="13.97" x2="25.4" y2="15.24" width="0.1524" layer="91"/>
+<wire x1="25.4" y1="15.24" x2="25.4" y2="38.1" width="0.1524" layer="91"/>
+<wire x1="25.4" y1="38.1" x2="93.98" y2="38.1" width="0.1524" layer="91"/>
 </segment>
 </net>
@@
 <pinref part="U$2" gate="G$1" pin="1"/>
 <wire x1="43.18" y1="55.88" x2="63.5" y2="55.88" width="0.1524" layer="91"/>
-<wire x1="63.5" y1="55.88" x2="63.5" y2="38.1" width="0.1524" layer="91"/>
-<wire x1="63.5" y1="38.1" x2="30.48" y2="38.1" width="0.1524" layer="91"/>
+<wire x1="63.5" y1="55.88" x2="63.5" y2="40.64" width="0.1524" layer="91"/>
+<wire x1="63.5" y1="40.64" x2="30.48" y2="40.64" width="0.1524" layer="91"/>
 <pinref part="U$1" gate="G$1" pin="4"/>
-<wire x1="30.48" y1="38.1" x2="30.48" y2="21.59" width="0.1524" layer="91"/>
-<wire x1="30.48" y1="21.59" x2="0" y2="21.59" width="0.1524" layer="91"/>
+<wire x1="0" y1="21.59" x2="17.78" y2="21.59" width="0.1524" layer="91"/>
+<wire x1="17.78" y1="21.59" x2="17.78" y2="40.64" width="0.1524" layer="91"/>
+<wire x1="17.78" y1="40.64" x2="30.48" y2="40.64" width="0.1524" layer="91"/>
 </segment>
 </net>
@@
 <wire x1="2.54" y1="63.5" x2="2.54" y2="57.15" width="0.1524" layer="91"/>
 <wire x1="2.54" y1="57.15" x2="0" y2="57.15" width="0.1524" layer="91"/>
-<pinref part="U$1" gate="G$1" pin="3"/>
-<wire x1="0" y1="24.13" x2="27.94" y2="24.13" width="0.1524" layer="91"/>
-<wire x1="27.94" y1="24.13" x2="27.94" y2="63.5" width="0.1524" layer="91"/>
+<pinref part="U$1" gate="G$1" pin="8"/>
+<wire x1="0" y1="11.43" x2="27.94" y2="11.43" width="0.1524" layer="91"/>
+<wire x1="27.94" y1="11.43" x2="27.94" y2="63.5" width="0.1524" layer="91"/>
 <wire x1="27.94" y1="63.5" x2="2.54" y2="63.5" width="0.1524" layer="91"/>
 <junction x="2.54" y="63.5"/>
 </segment>
 </net>
+<net name="N$3" class="0">
+<segment>
+<pinref part="U$1" gate="G$1" pin="6"/>
+<wire x1="0" y1="16.51" x2="22.86" y2="16.51" width="0.1524" layer="91"/>
+<wire x1="22.86" y1="16.51" x2="22.86" y2="20.32" width="0.1524" layer="91"/>
+<pinref part="R2" gate="G$1" pin="1"/>
+<wire x1="22.86" y1="20.32" x2="38.1" y2="20.32" width="0.1524" layer="91"/>
+</segment>
+</net>

Commit message: [update] コネクタをPHにして裏に部品を実装するようにした
Parts:
- removed U$1: PIN_HEADER_MALE_1X08_08P, 180118 Library by matsu:PIN_HEADER_MALE_1X08_08P
- removed U$2: PIN_HEADER_MALE_1X03_03P, 180118 Library by matsu:PIN_HEADER_MALE_1X03_03P
- removed U$3: PIN_HEADER_MALE_1X02_02P, 180118 Library by matsu:PIN_HEADER_MALE_1X02_02P
- added CN1: (no value), jst-ph:B8B-PH-K-S
- added CN2: (no value), jst-ph:B2B-PH-K-S
- added CN3: (no value), jst-ph:B3B-PH-K-S
Connections:
- net +3V3: now also CN1.1; no longer U$1.1
- net +5V: now also CN1.2, CN3.2; no longer U$1.2, U$2.2
- net GND: now also CN1.3, CN2.2, CN3.3; no longer U$1.3, U$2.3, U$3.2
- net N$3: now also CN1.6; no longer U$1.6
- net N$4: now also CN1.5; no longer U$1.5
- net N$5: now also CN1.7; no longer U$1.7
- net N$6: now also CN1.8, CN2.1; no longer U$1.8, U$3.1
- net N$8: now also CN1.4, CN3.1; no longer U$1.4, U$2.1
Changed lines of the file:
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@@
 <?xml version="1.0" encoding="utf-8"?>
 <!DOCTYPE eagle SYSTEM "eagle.dtd">
-<eagle version="9.1.1">
+<eagle version="9.1.3">
 <drawing>
 <settings>
@@
 <parts>
 <part name="SW1" library="TVGP01-G73BB" deviceset="TVGP01-G73BB" device=""/>
-<part name="U$2" library="180118 Library by matsu" deviceset="PIN_HEADER_MALE_1X03_03P" device=""/>
 <part name="LED1" library="180118 Library by matsu" deviceset="LED" device="5MM"/>
 <part name="LED2" library="180118 Library by matsu" deviceset="LED" device="5MM"/>
@@
 <part name="+3V1" library="180118 Library by matsu" deviceset="+3V3" device=""/>
 <part name="+3V2" library="180118 Library by matsu" deviceset="+3V3" device=""/>
-<part name="U$1" library="180118 Library by matsu" deviceset="PIN_HEADER_MALE_1X08_08P" device=""/>
 <part name="R3" library="180118 Library by matsu" deviceset="R-EU_" device="0204/7"/>
 <part name="GND4" library="180118 Library by matsu" deviceset="GND" device=""/>
 <part name="GND5" library="180118 Library by matsu" deviceset="GND" device=""/>
-<part name="U$3" library="180118 Library by matsu" deviceset="PIN_HEADER_MALE_1X02_02P" device=""/>
 <part name="+3V3" library="180118 Library by matsu" deviceset="+3V3" device=""/>
 <part name="GND6" library="180118 Library by matsu" deviceset="GND" device=""/>
 <part name="R4" library="180118 Library by matsu" deviceset="R-EU_" device="0204/7"/>
+<part name="CN1" library="jst-ph" deviceset="B8B-PH-*" device="K-S"/>
+<part name="CN2" library="jst-ph" deviceset="B2B-PH-*" device="K-S"/>
+<part name="CN3" library="jst-ph" deviceset="B3B-PH-*" device="K-S"/>
 </parts>
 <sheets>
@@
 <instances>
 <instance part="SW1" gate="G$1" x="101.6" y="53.34" rot="R270"/>
-<instance part="U$2" gate="G$1" x="38.1" y="53.34" rot="R270"/>
 <instance part="LED1" gate="G$1" x="55.88" y="30.48" rot="R90"/>
 <instance part="LED2" gate="G$1" x="55.88" y="20.32" rot="R90"/>
@@
 <instance part="+3V1" gate="G$1" x="7.62" y="40.64"/>
 <instance part="+3V2" gate="G$1" x="78.74" y="66.04"/>
-<instance part="U$1" gate="G$1" x="-5.08" y="20.32" rot="R270"/>
 <instance part="R3" gate="G$1" x="86.36" y="53.34"/>
 <instance part="GND4" gate="1" x="114.3" y="45.72"/>
 <instance part="GND5" gate="1" x="50.8" y="45.72"/>
-<instance part="U$3" gate="G$1" x="-5.08" y="55.88" rot="R270"/>
 <instance part="+3V3" gate="G$1" x="20.32" y="73.66"/>
 <instance part="GND6" gate="1" x="5.08" y="48.26"/>
 <instance part="R4" gate="G$1" x="10.16" y="68.58"/>
+<instance part="CN1" gate="G$1" x="-5.08" y="22.86"/>
+<instance part="CN2" gate="G$1" x="12.7" y="58.42"/>
+<instance part="CN3" gate="G$1" x="55.88" y="53.34"/>
 </instances>
 <busses>
@@
 <net name="+5V" class="1">
 <segment>
-<pinref part="U$2" gate="G$1" pin="2"/>
 <pinref part="P+2" gate="1" pin="+5V"/>
-<wire x1="43.18" y1="53.34" x2="50.8" y2="53.34" width="0.1524" layer="91"/>
 <wire x1="50.8" y1="53.34" x2="50.8" y2="63.5" width="0.1524" layer="91"/>
-</segment>
-<segment>
-<pinref part="U$1" gate="G$1" pin="2"/>
+<pinref part="CN3" gate="G$1" pin="2"/>
+<wire x1="55.88" y1="53.34" x2="50.8" y2="53.34" width="0.1524" layer="91"/>
+</segment>
+<segment>
 <pinref part="P+1" gate="1" pin="+5V"/>
-<wire x1="0" y1="26.67" x2="15.24" y2="26.67" width="0.1524" layer="91"/>
-<wire x1="15.24" y1="26.67" x2="15.24" y2="38.1" width="0.1524" layer="91"/>
+<wire x1="15.24" y1="38.1" x2="15.24" y2="27.94" width="0.1524" layer="91"/>
+<pinref part="CN1" gate="G$1" pin="2"/>
+<wire x1="15.24" y1="27.94" x2="-5.08" y2="27.94" width="0.1524" layer="91"/>
 </segment>
 </net>
@@
 </segment>
 <segment>
-<pinref part="U$1" gate="G$1" pin="1"/>
+<pinref part="CN1" gate="G$1" pin="1"/>
 <pinref part="+3V1" gate="G$1" pin="+3V3"/>
-<wire x1="0" y1="29.21" x2="7.62" y2="29.21" width="0.1524" layer="91"/>
-<wire x1="7.62" y1="29.21" x2="7.62" y2="38.1" width="0.1524" layer="91"/>
+<wire x1="-5.08" y1="30.48" x2="7.62" y2="30.48" width="0.1524" layer="91"/>
+<wire x1="7.62" y1="30.48" x2="7.62" y2="38.1" width="0.1524" layer="91"/>
 </segment>
 </net>
@@
 </segment>
 <segment>
-<pinref part="U$2" gate="G$1" pin="3"/>
 <pinref part="GND5" gate="1" pin="GND"/>
-<wire x1="43.18" y1="50.8" x2="50.8" y2="50.8" width="0.1524" layer="91"/>
 <wire x1="50.8" y1="50.8" x2="50.8" y2="48.26" width="0.1524" layer="91"/>
-</segment>
-<segment>
-<pinref part="U$3" gate="G$1" pin="2"/>
+<pinref part="CN3" gate="G$1" pin="3"/>
+<wire x1="55.88" y1="50.8" x2="50.8" y2="50.8" width="0.1524" layer="91"/>
+</segment>
+<segment>
+<pinref part="GND3" gate="1" pin="GND"/>
+<wire x1="30.48" y1="24.13" x2="30.48" y2="22.86" width="0.1524" layer="91"/>
+<pinref part="CN1" gate="G$1" pin="3"/>
+<wire x1="30.48" y1="22.86" x2="30.48" y2="5.08" width="0.1524" layer="91"/>
+<wire x1="-5.08" y1="25.4" x2="30.48" y2="25.4" width="0.1524" layer="91"/>
+<wire x1="30.48" y1="25.4" x2="30.48" y2="22.86" width="0.1524" layer="91"/>
+</segment>
+<segment>
+<pinref part="CN2" gate="G$1" pin="2"/>
 <pinref part="GND6" gate="1" pin="GND"/>
-<wire x1="0" y1="54.61" x2="5.08" y2="54.61" width="0.1524" layer="91"/>
-<wire x1="5.08" y1="54.61" x2="5.08" y2="50.8" width="0.1524" layer="91"/>
-</segment>
-<segment>
-<pinref part="U$1" gate="G$1" pin="3"/>
-<pinref part="GND3" gate="1" pin="GND"/>
-<wire x1="0" y1="24.13" x2="30.48" y2="24.13" width="0.1524" layer="91"/>
-<wire x1="30.48" y1="24.13" x2="30.48" y2="5.08" width="0.1524" layer="91"/>
+<wire x1="12.7" y1="55.88" x2="5.08" y2="55.88" width="0.1524" layer="91"/>
+<wire x1="5.08" y1="55.88" x2="5.08" y2="50.8" width="0.1524" layer="91"/>
 </segment>
 </net>
@@
 <wire x1="38.1" y1="30.48" x2="35.56" y2="30.48" width="0.1524" layer="91"/>
 <wire x1="35.56" y1="30.48" x2="33.02" y2="30.48" width="0.1524" layer="91"/>
-<pinref part="U$1" gate="G$1" pin="5"/>
-<wire x1="0" y1="19.05" x2="20.32" y2="19.05" width="0.1524" layer="91"/>
-<wire x1="20.32" y1="19.05" x2="20.32" y2="30.48" width="0.1524" layer="91"/>
 <wire x1="20.32" y1="30.48" x2="33.02" y2="30.48" width="0.1524" layer="91"/>
+<pinref part="CN1" gate="G$1" pin="5"/>
+<wire x1="-5.08" y1="20.32" x2="20.32" y2="20.32" width="0.1524" layer="91"/>
+<wire x1="20.32" y1="20.32" x2="20.32" y2="30.48" width="0.1524" layer="91"/>
 </segment>
 </net>
@@
 <wire x1="93.98" y1="53.34" x2="96.52" y2="53.34" width="0.1524" layer="91"/>
 <junction x="93.98" y="53.34"/>
-<pinref part="U$1" gate="G$1" pin="7"/>
 <wire x1="93.98" y1="38.1" x2="93.98" y2="53.34" width="0.1524" layer="91"/>
-<wire x1="0" y1="13.97" x2="25.4" y2="13.97" width="0.1524" layer="91"/>
-<wire x1="25.4" y1="13.97" x2="25.4" y2="15.24" width="0.1524" layer="91"/>
+<wire x1="25.4" y1="38.1" x2="93.98" y2="38.1" width="0.1524" layer="91"/>
+<pinref part="CN1" gate="G$1" pin="7"/>
+<wire x1="-5.08" y1="15.24" x2="25.4" y2="15.24" width="0.1524" layer="91"/>
 <wire x1="25.4" y1="15.24" x2="25.4" y2="38.1" width="0.1524" layer="91"/>
-<wire x1="25.4" y1="38.1" x2="93.98" y2="38.1" width="0.1524" layer="91"/>
 </segment>
 </net>
 <net name="N$8" class="0">
 <segment>
-<pinref part="U$2" gate="G$1" pin="1"/>
-<wire x1="43.18" y1="55.88" x2="63.5" y2="55.88" width="0.1524" layer="91"/>
-<wire x1="63.5" y1="55.88" x2="63.5" y2="40.64" width="0.1524" layer="91"/>
-<wire x1="63.5" y1="40.64" x2="30.48" y2="40.64" width="0.1524" layer="91"/>
-<pinref part="U$1" gate="G$1" pin="4"/>
-<wire x1="0" y1="21.59" x2="17.78" y2="21.59" width="0.1524" layer="91"/>
-<wire x1="17.78" y1="21.59" x2="17.78" y2="40.64" width="0.1524" layer="91"/>
 <wire x1="17.78" y1="40.64" x2="30.48" y2="40.64" width="0.1524" layer="91"/>
+<pinref part="CN3" gate="G$1" pin="1"/>
+<wire x1="55.88" y1="55.88" x2="43.18" y2="55.88" width="0.1524" layer="91"/>
+<wire x1="43.18" y1="55.88" x2="43.18" y2="43.18" width="0.1524" layer="91"/>
+<wire x1="43.18" y1="43.18" x2="43.18" y2="40.64" width="0.1524" layer="91"/>
+<wire x1="43.18" y1="40.64" x2="30.48" y2="40.64" width="0.1524" layer="91"/>
+<pinref part="CN1" gate="G$1" pin="4"/>
+<wire x1="-5.08" y1="22.86" x2="17.78" y2="22.86" width="0.1524" layer="91"/>
+<wire x1="17.78" y1="22.86" x2="17.78" y2="40.64" width="0.1524" layer="91"/>
 </segment>
 </net>
@@
 <wire x1="5.08" y1="68.58" x2="2.54" y2="68.58" width="0.1524" layer="91"/>
 <wire x1="2.54" y1="68.58" x2="2.54" y2="63.5" width="0.1524" layer="91"/>
-<pinref part="U$3" gate="G$1" pin="1"/>
-<wire x1="2.54" y1="63.5" x2="2.54" y2="57.15" width="0.1524" layer="91"/>
-<wire x1="2.54" y1="57.15" x2="0" y2="57.15" width="0.1524" layer="91"/>
-<pinref part="U$1" gate="G$1" pin="8"/>
-<wire x1="0" y1="11.43" x2="27.94" y2="11.43" width="0.1524" layer="91"/>
-<wire x1="27.94" y1="11.43" x2="27.94" y2="63.5" width="0.1524" layer="91"/>
 <wire x1="27.94" y1="63.5" x2="2.54" y2="63.5" width="0.1524" layer="91"/>
+<pinref part="CN2" gate="G$1" pin="1"/>
+<wire x1="12.7" y1="58.42" x2="2.54" y2="58.42" width="0.1524" layer="91"/>
+<wire x1="2.54" y1="58.42" x2="2.54" y2="63.5" width="0.1524" layer="91"/>
 <junction x="2.54" y="63.5"/>
+<wire x1="27.94" y1="63.5" x2="27.94" y2="12.7" width="0.1524" layer="91"/>
+<pinref part="CN1" gate="G$1" pin="8"/>
+<wire x1="27.94" y1="12.7" x2="-5.08" y2="12.7" width="0.1524" layer="91"/>
 </segment>
 </net>
 <net name="N$3" class="0">
 <segment>
-<pinref part="U$1" gate="G$1" pin="6"/>
-<wire x1="0" y1="16.51" x2="22.86" y2="16.51" width="0.1524" layer="91"/>
-<wire x1="22.86" y1="16.51" x2="22.86" y2="20.32" width="0.1524" layer="91"/>
 <pinref part="R2" gate="G$1" pin="1"/>
 <wire x1="22.86" y1="20.32" x2="38.1" y2="20.32" width="0.1524" layer="91"/>
-</segment>
-</net>
+<pinref part="CN1" gate="G$1" pin="6"/>
+<wire x1="-5.08" y1="17.78" x2="22.86" y2="17.78" width="0.1524" layer="91"/>
+<wire x1="22.86" y1="17.78" x2="22.86" y2="20.32" width="0.1524" layer="91"/>
+</segment>
+</net>
